File: src/schematics/ScouseTom_SwitchNetwork/SwitchBoard.sch (EAGLE design)
At the start: 86 parts, among them IC2 LT1763CDE-5, U1 ADUM1410ARWZ, U2 MCP73831, U3 TPS61090RSAR, X1 DSUB _T, X2 DSUB_B, X3 USB-MICROB

Commit message: SwitchNetwork Finished. Gerber/BOM/P&P generated
Parts:
- removed C28: 2.2uF, resistor:C-EUC0805
- removed DSUB1: CTR_OUT, con-subd:M09HP
- removed DSUB2: CTR_ARD, con-subd:F09HP
- removed JP12: LiPoIN, SparkFun:M02PTH
- removed NSW1, PSW1: ADG714BRUZ, Analog Devices_By_element14_Batch_1:ADG714BRUZ
- removed ON/OFF: (no value), pinhead:PINHD-1X2
- added C27: 1uF, resistor:C-EUC0805
- added JP6: Shld, pinhead:PINHD-1X2
- added JP7: DCHN, pinhead:PINHD-2X9
- added JP8: CS_IN+, pinhead:PINHD-1X1
- added U12: ADUM1410ARWZ, ADI-Phase-2:ADUM1410ARWZ
- added U4: TPS61090RSAR, Adafruit PowerBoost 500C:VREG_TPS6103XSPARKFUNVERSION
- added X4: DSUB _T, con-subd:F37HP
- added X5: DSUB_B, con-subd:M37HP
- C1, C3: value .1uF -> 10uF
- C10: value 10uF -> 100uF; device resistor:C-EUC0805 -> rcl:CPOL-EUCT6032
- C11: value 0.1uF -> 10uF
- C14: value 0.1uF -> 0.01uF
- C15: value 0.1uF -> 100uF; device resistor:C-EUC0805 -> rcl:CPOL-EUCT6032
- C16: value .1uF -> 0.1uF
- C17, C4: value 1uF -> 0.1uF
- C18: value 0.1uF -> .1uF
- C19: value .1uF -> 1uF
- C2: value 1uF -> 10uF
- C20: value 1uF -> .1uF
- C21, C25: value 10uF -> 1uF
- C22: value 100uF -> 0.1uF; device rcl:CPOL-EUCT6032 -> resistor:C-EUC0805
- C23: value 0.01uF -> 0.1uF
- C24: value 10uF -> .1uF
- C26: value 100uF -> .1uF; device rcl:CPOL-EUCT6032 -> resistor:C-EUC0805
- C9: value 0.1uF -> 2.2uF
- JP1: value (none) -> IN; device pinhead:PINHD-1X2 -> SparkFun:M02PTH
- JP2: value LiPo -> LiPoIN; device SparkFun:M02-JST-2MM-SMT -> SparkFun:M02PTH
- JP3: value (none) -> LiPo; device pinhead:PINHD-1X2 -> SparkFun:M02-JST-2MM-SMT
- JP4: value (none) -> PWR
- JP5: value (none) -> Shld; device pinhead:PINHD-2X9 -> pinhead:PINHD-1X2
- JP9: value IN -> CS_IN-; device SparkFun:M02PTH -> pinhead:PINHD-1X1
- LED4: value GREEN -> RED
- R1: value 10k -> 470
- R10: value 10k -> 200k
- R11: value 10M -> 1k
- R12: value 10M -> 10k
- R13, R17, R21: value 1k -> 10k
- R14: value 470 -> 4.7k
- R15: value 2k -> 47k
- R16: value 1.8M -> 1k
- R18: value 200k -> 10k
- R19: value 82k -> 10k
- R2: value 10k -> 1k
- R20: value 2M -> 10k
- R22: value 4.7k -> 10k
- R23: value 360k -> 10M
- R24: value 47k -> 10M
- R3: value 10k -> 2k
- R4: value 10k -> 2M
- R5: value 10k -> 360k
- R8: value 10k -> 1.8M
- R9: value 10k -> 82k
- T1: value (none) -> PNP
- U1: value ADUM1410ARWZ -> MCP73831; device ADI-Phase-2:ADUM1410ARWZ -> SparkFun-PowerIC:MCP73831
- U2: value MCP73831 -> ADG714BRUZ; device SparkFun:MCP73831 -> Analog Devices_By_element14_Batch_1:ADG714BRUZ
- U3: value TPS61090RSAR -> ADG714BRUZ; device Adafruit PowerBoost 500C:VREG_TPS6103XSPARKFUNVERSION -> Analog Devices_By_element14_Batch_1:ADG714BRUZ
- X1: value DSUB _T -> USB-MICROB; device con-subd:F37HP -> SparkFun:USB-MICROB
- X2: value DSUB_B -> CTR_ARD; device con-subd:M37HP -> con-subd:F09HP
- X3: value USB-MICROB -> CTR_OUT; device SparkFun:USB-MICROB -> con-subd:M09HP
- renumbered CHRG to LED1, DSUB3 to X6, FULL to LED2, IC2 to U8, L2 to L1, LBO to LED4, NSW2 to U6, NSW3 to U9, NSW4 to U11, NSW5 to U14, PSW2 to U5, PSW3 to U7, PSW4 to U10, PSW5 to U13, PWR to LED3, U$1 to U15
Connections:
- removed net N$2: LED1.C, R14.2
- new net CHRG: LED1.C, R1.2
- net +5V: now also C21.1, C26.1, C27.1, U12.VDD1, X2.9; no longer C19.1, C3.1, C4.1, DSUB2.9, U1.VDD1
- net 5VIN: now also C1.1, JP1.1, U1.VIN, X1.VBUS; no longer C10.1, JP9.1, U2.VIN, X3.VBUS
- net AGND: now also C10.-, C11.2, C15.-, C16.1, C17.1, C18.2, C19.2, C22.1, C23.1, C3.2, C4.2, JP1.2, JP2.2, JP5.1, JP6.2, JP7.3, R10.1, R11.2, R24.1, R3.1, R5.1, U1.VSS, U12.CTRL2, U12.GND2, U12.GND2_2, U2.GND, U3.VSS, U4.GND, U4.PGND, U4.SYNC, X1.GND, X3.6; no longer C10.2, C11.1, C14.1, C15.1, C16.2, C17.2, C18.1, C21.2, C22.-, C26.-, C28.2, DSUB1.6, JP12.2, JP2.1, JP4.2, JP5.3, JP9.2, NSW1.GND, NSW1.VSS, PSW1.GND, PSW1.VSS, R11.1, R12.1, R15.1, R17.2, R18.1, U1.CTRL2, U1.GND2, U1.GND2_2, U3.PGND, U3.SYNC, X3.GND
- net DIN+: now also JP7.7, U12.VOB, U2.DIN; no longer JP5.7, PSW1.DIN, U1.VOB
- net DIN+2: now also R6.1, U2.DOUT; no longer PSW1.DOUT, R1.1
- net DIN+3: now also R12.1; no longer R2.1
- net DIN+4: now also R17.1; no longer R3.1
- net DIN+5: now also R19.1; no longer R4.1
- net DIN+_DCHN: now also JP7.8; no longer JP5.8
- net DIN+_IN: now also U12.VIB, X2.3; no longer DSUB2.3, U1.VIB
- net DIN-: now also JP7.9, U12.VOC, U3.DIN; no longer JP5.9, NSW1.DIN, U1.VOC
- net DIN-2: now also R7.1, U3.DOUT; no longer NSW1.DOUT, R6.1
- net DIN-3: now also R13.1; no longer R7.1
- net DIN-4: now also R18.1; no longer R8.1
- net DIN-5: now also R20.1; no longer R9.1
- net DIN-_DCHN: now also JP7.10; no longer JP5.10
- net DIN-_IN: now also U12.VIC, X2.7; no longer DSUB2.7, U1.VIC
- net DOUT+: now also R21.1, X3.3; no longer DSUB1.3, R5.1
- net DOUT-: now also R22.1, X3.7; no longer DSUB1.7, R10.1
- net GND: now also C21.2, C26.2, C27.2, U12.DISABLE, U12.GND1, U12.GND1_2, X2.6; no longer C19.2, C3.2, C4.2, DSUB2.6, U1.DISABLE, U1.GND1, U1.GND1_2
- net GND_DCHN: now also JP7.4; no longer JP5.4
- net IN+: now also JP8.1, U2.D1, U2.D2, U2.D3, U2.D4, U2.D5, U2.D6, U2.D7, U2.D8; no longer JP1.1, PSW1.D1, PSW1.D2, PSW1.D3, PSW1.D4, PSW1.D5, PSW1.D6, PSW1.D7, PSW1.D8
- net IN-: now also JP9.1, U3.D1, U3.D2, U3.D3, U3.D4, U3.D5, U3.D6, U3.D7, U3.D8; no longer JP1.2, NSW1.D1, NSW1.D2, NSW1.D3, NSW1.D4, NSW1.D5, NSW1.D6, NSW1.D7, NSW1.D8
- net LBO: now also R14.1, U4.LBO; no longer R22.1, U3.LBO
- net LB_REF: now also R4.1, R5.2, U4.LBI; no longer R20.1, R23.2, U3.LBI
- net N$10: now also JP5.2, X3.G1, X3.G2; no longer DSUB1.G1, DSUB1.G2, JP3.2
- net N$11: now also R14.2, R15.1; no longer R22.2, R24.1
- net N$12: now also JP6.1; no longer JP4.1
- net N$3: now also C14.1; no longer C23.1
- net N$4: now also C14.2; no longer C23.2
- net N$5: now also R2.2; no longer R13.2
- net N$6: now also R8.1, R9.2; no longer R16.1, R19.2
- net N$7: now also R11.1; no longer R17.1
- net N$8: now also R16.1; no longer R21.1
- net N$9: now also R16.2; no longer R21.2
- net OUT_1: now also U2.S1, U3.S1, X4.1, X5.1; no longer NSW1.S1, PSW1.S1, X1.1, X2.1
- net OUT_10: now also X4.10, X5.10; no longer X1.10, X2.10
- net OUT_11: now also X4.11, X5.11; no longer X1.11, X2.11
- net OUT_12: now also X4.12, X5.12; no longer X1.12, X2.12
- net OUT_13: now also X4.13, X5.13; no longer X1.13, X2.13
- net OUT_14: now also X4.14, X5.14; no longer X1.14, X2.14
- net OUT_15: now also X4.15, X5.15; no longer X1.15, X2.15
- net OUT_16: now also X4.16, X5.16; no longer X1.16, X2.16
- net OUT_17: now also X4.17, X5.17; no longer X1.17, X2.17
- net OUT_18: now also X4.18, X5.18; no longer X1.18, X2.18
- net OUT_19: now also X4.19, X5.19; no longer X1.19, X2.19
- net OUT_2: now also U2.S2, U3.S2, X4.2, X5.2; no longer NSW1.S2, PSW1.S2, X1.2, X2.2
- net OUT_20: now also X4.20, X5.20; no longer X1.20, X2.20
- net OUT_21: now also X4.21, X5.21; no longer X1.21, X2.21
- net OUT_22: now also X4.22, X5.22; no longer X1.22, X2.22
- net OUT_23: now also X4.23, X5.23; no longer X1.23, X2.23
- net OUT_24: now also X4.24, X5.24; no longer X1.24, X2.24
- net OUT_25: now also X4.25, X5.25; no longer X1.25, X2.25
- net OUT_26: now also X4.26, X5.26; no longer X1.26, X2.26
- net OUT_27: now also X4.27, X5.27; no longer X1.27, X2.27
- net OUT_28: now also X4.28, X5.28; no longer X1.28, X2.28
- net OUT_29: now also X4.29, X5.29; no longer X1.29, X2.29
- net OUT_3: now also U2.S3, U3.S3, X4.3, X5.3; no longer NSW1.S3, PSW1.S3, X1.3, X2.3
- net OUT_30: now also X4.30, X5.30; no longer X1.30, X2.30
- net OUT_31: now also X4.31, X5.31; no longer X1.31, X2.31
- net OUT_32: now also X4.32, X5.32; no longer X1.32, X2.32
- net OUT_33: now also X4.33, X5.33; no longer X1.33, X2.33
- net OUT_34: now also X4.34, X5.34; no longer X1.34, X2.34
- net OUT_35: now also X4.35, X5.35; no longer X1.35, X2.35
- net OUT_36: now also X4.36, X5.36; no longer X1.36, X2.36
- net OUT_37: now also X4.37, X5.37; no longer X1.37, X2.37
- net OUT_4: now also U2.S4, U3.S4, X4.4, X5.4; no longer NSW1.S4, PSW1.S4, X1.4, X2.4
- net OUT_5: now also U2.S5, U3.S5, X4.5, X5.5; no longer NSW1.S5, PSW1.S5, X1.5, X2.5
- net OUT_6: now also U2.S6, U3.S6, X4.6, X5.6; no longer NSW1.S6, PSW1.S6, X1.6, X2.6
- net OUT_7: now also U2.S7, U3.S7, X4.7, X5.7; no longer NSW1.S7, PSW1.S7, X1.7, X2.7
- net OUT_8: now also U2.S8, U3.S8, X4.8, X5.8; no longer NSW1.S8, PSW1.S8, X1.8, X2.8
- net OUT_9: now also X4.9, X5.9; no longer X1.9, X2.9
- net PROG: now also R3.2, U1.PROG; no longer R15.2, U2.PROG
- net RESET_DCHN: now also JP7.14; no longer JP5.14
- net RESET_IN: now also X2.8; no longer DSUB2.8
- net SCLK: now also JP7.11, U12.VOD, U2.SCLK, U3.SCLK, X3.2; no longer DSUB1.2, JP5.11, NSW1.SCLK, PSW1.SCLK, U1.VOD
- net SCLK_DCHN: now also JP7.12; no longer JP5.12
- net SCLK_IN: now also U12.VID, X2.2; no longer DSUB2.2, U1.VID
- net STAT: now also R1.1, R2.1, U1.STAT; no longer R13.1, R14.1, U2.STAT
- net SW: now also U4.SW; no longer U3.SW
- net SYNC_DCHN: now also JP7.6; no longer JP5.6
- net SYNC_IN: now also U12.VIA, X2.4; no longer DSUB2.4, U1.VIA
- net TEST_1: now also JP7.15, R23.2, X3.5; no longer DSUB1.5, JP5.15, R11.2
- net TEST_1_DCHN: now also JP7.16; no longer JP5.16
- net TEST_1_IN: now also X2.5; no longer DSUB2.5
- net TEST_2: now also JP7.17, R24.2, X3.1; no longer DSUB1.1, JP5.17, R12.2
- net TEST_2_DCHN: now also JP7.18; no longer JP5.18
- net TEST_2_IN: now also X2.1; no longer DSUB2.1
- net VBATT_A: now also C2.1, JP2.1, JP3.2, JP4.1, U1.VBAT; no longer C24.1, JP12.1, JP2.2, ON/OFF.1, U2.VBAT
- net VBATT_B: now also C3.1, C4.1, JP4.2, R15.2, R4.2, U4.EN, U4.VBAT; no longer C25.1, C9.1, ON/OFF.2, R20.2, R24.2, U3.EN, U3.VBAT
- net VDD: now also C15.+, C16.2, C17.2, C18.1, C19.1, C22.2, C23.2, C24.1, C25.1, JP7.1, R12.2, R13.2, R17.2, R18.2, R19.2, R20.2, R21.2, R22.2, U12.VDD2, U2.VDD, U3.VDD, X3.9; no longer C1.1, C11.2, C14.2, C15.2, C16.1, C17.1, C18.2, C2.1, C22.+, DSUB1.9, JP5.1, NSW1.VDD, PSW1.VDD, R1.2, R10.2, R2.2, R3.2, R4.2, R5.2, R8.2, R9.2, U1.VDD2
- net VDD_DCHN: now also JP7.2; no longer JP5.2
- net VREG: now also C10.+, C11.1, C9.1, R8.2, U4.VOUT; no longer C21.1, C26.+, C28.1, R16.2, U3.VOUT
- net VSET: now also R10.2, R9.1, U4.FB; no longer R18.2, R19.1, U3.FB
- net ~RESET: now also JP7.13, U2.~RESET, U3.~RESET, X3.8; no longer DSUB1.8, JP5.13, NSW1.~RESET, PSW1.~RESET
- net ~SYNC: now also JP7.5, U12.VOA, U2.~SYNC, U3.~SYNC, X3.4; no longer DSUB1.4, JP5.5, NSW1.~SYNC, PSW1.~SYNC, U1.VOA
Other:
- moved on the sheet: C1, C11, C12, C13, C14, C16, C17, C18, C19, C2, C20, C21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
