File: src/schematics/Output_Impedance_Tester/OutputZTester.sch (EAGLE design)
At the start: 0 parts

Commit message: Finished sim of TIA and Droop circuit. Started PCB
Parts:
- added C1, C4: 2.2uF, rcl:C-EUC0402
- added C10, C11, C12, C2, C5, C7, C8, C9: 0.1uF, rcl:C-EUC0402
- added C3, C6: 10nF, rcl:C-EUC0402
- added D1, D2: (no value), diode:DIODE-DO-214AC
- added JP1: PWR_IN, pinhead:PINHD-1X3/90
- added JP2: (no value), pinhead:PINHD-1X3/90
- added R1, R10, R11, R12, R13, R14, R15, R16, R17, R18, R19, R2, R20, R21, R22, R23, R24, R25, R27, R28, R29, R3, R30, R31, R4, R5, R6, R7, R8, R9: (no value), rcl:R-EU_R0402
- added TP1, TP2, TP3, TP4, TP5: TPSB1,27, testpad:TPSB1,27
- added U1, U3, U4, U5: ADG801BRTZ-REEL7, Analog Devices_By_element14_Batch_1:ADG801BRTZ-REEL7
- added U2: ADA4552-2ARM, ScouseTomLib:ADA4552-2ARM
Connections:
- new net AGND: C1.2, C10.1, C11.1, C12.1, C2.2, C3.2, C4.2, C5.2, C6.2, C7.1, C8.2, C9.1, D1.A, D2.C, JP1.2, JP2.3, R7.1, U1.GND, U1.NC, U1.S, U3.GND, U3.NC, U3.S, U4.GND, U4.NC, U4.S, U5.GND, U5.NC, U5.S
- new net N$10: R10.1, R11.1
- new net N$11: R12.1, R13.1
- new net N$12: R13.2, R14.2
- new net N$13: R14.1, R15.1
- new net N$14: R15.2, U3.D
- new net N$15: R16.2, R17.2
- new net N$16: R17.1, R18.1
- new net N$17: R18.2, R19.2
- new net N$18: R19.1, R20.1
- new net N$19: R20.2, U4.D
- new net N$2: R1.2, R2.2
- new net N$20: R21.2, R22.2
- new net N$21: R22.1, R23.1
- new net N$22: R23.2, R24.2
- new net N$23: R24.1, R25.1
- new net N$24: R25.2, U5.D
- new net N$26: R27.2, R28.2
- new net N$27: R28.1, R29.1
- new net N$28: R29.2, R30.2
- new net N$29: R30.1, R31.1
- new net N$3: R2.1, R3.1
- new net N$31: R31.2, U1.D
- new net N$4: R3.2, R5.2
- new net N$5: R5.1, R6.1
- new net N$6: R12.2, R4.2
- new net N$7: R7.2, R8.2
- new net N$8: R8.1, R9.1
- new net N$9: R10.2, R9.2
- new net SW1_PARA: U1.IN
- new net SW2_PARA: U3.IN
- new net SW3_PARA: U4.IN
- new net SW4_PARA: U5.IN
- new net V+: C1.1, C10.2, C11.2, C12.2, C2.1, C3.1, C7.2, C9.2, D1.C, JP1.1, TP1.PP, U1.VDD, U2.V+, U3.VDD, U4.VDD, U5.VDD
- new net V-: C4.1, C5.1, C6.1, C8.1, D2.A, JP1.3, TP2.PP, U2.V-
- new net VAMP_PARA: JP2.2, R1.1, TP5.PP, U2.OUT_B
- new net VBUFF: JP2.1, TP4.PP, U2.+IN_B, U2.-IN_A, U2.OUT_A
- new net VF_PARA: R11.2, R6.2, U2.-IN_B
- new net VLOAD_PARA: R16.1, R21.1, R27.1, R4.1, TP3.PP, U2.+IN_A
