File: src/schematics/Output_Impedance_Tester/OutputZTester.sch (EAGLE design)
At the start: 56 parts, among them U1 ADG801BRTZ-REEL7, U2 ADA4552-2ARM, U3 ADG801BRTZ-REEL7, U4 ADG801BRTZ-REEL7, U5 ADG801BRTZ-REEL7

Commit message: Basic layout for both circuits done
Parts:
- added C13, C14, C16, C17, C18, C19: 0.1uF, rcl:C-EUC0402
- added C15: 2.2nF, rcl:C-EUC0402
- added JP3: (no value), pinhead:PINHD-1X5/90
- added JP4: PWR_IN, pinhead:PINHD-1X2/90
- added JP5: Source, pinhead:PINHD-1X1
- added JP6: Sink, pinhead:PINHD-1X1
- added JP7: (no value), pinhead:PINHD-1X1
- added R26, R32, R33, R34, R35, R36, R37, R38, R39, R40, R41, R42, R43, R44, R45, R46, R47, R48, R49, R50, R51, R52, R53, R54, R55, R56, R57, R58, R59, R60, R61, R62, R63, R64, R65: (no value), rcl:R-EU_R0402
- added U10, U7, U8, U9: ADG801BRTZ-REEL7, Analog Devices_By_element14_Batch_1:ADG801BRTZ-REEL7
- added U6: ADA4552-2ARM, ScouseTomLib:ADA4552-2ARM
- D1, D2: value (none) -> 1N4148W-7-F; device diode:DIODE-DO-214AC -> diode:DIODE-SOD123
- JP1: device pinhead:PINHD-1X3/90 -> pinhead:PINHD-1X2/90
Connections:
- new net N$1: R26.2, R32.2
- new net N$25: R32.1, R33.1
- new net N$30: R33.2, R34.2
- new net N$32: R34.1, R35.1
- new net N$33: R36.2, R37.2
- new net N$34: R37.1, R38.1
- new net N$35: R38.2, R39.2
- new net N$36: R39.1, R40.1
- new net N$37: R41.2, R42.2
- new net N$38: R42.1, R43.1
- new net N$39: R43.2, R44.2
- new net N$40: R44.1, R45.1
- new net N$41: R46.2, R47.2
- new net N$42: R47.1, R48.1
- new net N$43: R48.2, R49.2
- new net N$44: R49.1, R50.1
- new net N$46: R50.2, U7.S
- new net N$47: R51.2, R52.2
- new net N$48: R52.1, R53.1
- new net N$49: R53.2, R54.2
- new net N$50: R54.1, R55.1
- new net N$51: R55.2, U8.S
- new net N$52: R56.2, R57.2
- new net N$53: R57.1, R58.1
- new net N$54: R58.2, R59.2
- new net N$55: R59.1, R60.1
- new net N$56: R60.2, U9.S
- new net N$57: R61.2, R62.2
- new net N$58: R62.1, R63.1
- new net N$59: R63.2, R64.2
- new net N$60: R64.1, R65.1
- new net N$61: R65.2, U10.S
- new net SOURCE_TIA: JP7.1, U10.D, U7.D, U8.D, U9.D
- new net SW1_TIA: U10.IN
- new net SW2_TIA: U7.IN
- new net SW3_TIA: U8.IN
- new net SW4_TIA: U9.IN
- new net VAMP_TIA: R26.1, U6.OUT_A
- new net VF_TIA: R35.2, R40.2, U6.-IN_A
- new net VLOAD_TIA: C15.1, R41.1, R46.1, R51.1, R56.1, R61.1, U6.-IN_B
- new net VOUT_TIA: C15.2, R45.2, U6.+IN_A, U6.OUT_B
- net AGND: now also C13.1, C14.2, C16.1, C17.1, C18.1, C19.1, JP1.1, JP3.5, JP4.1, JP6.1, R36.1, U10.GND, U10.NC, U6.+IN_B, U7.GND, U7.NC, U8.GND, U8.NC, U9.GND, U9.NC; no longer JP1.2
- net SW1_PARA: now also JP3.1
- net SW2_PARA: now also JP3.2
- net SW3_PARA: now also JP3.3
- net SW4_PARA: now also JP3.4
- net V+: now also C13.2, C16.2, C17.2, C18.2, C19.2, JP1.2, U10.VDD, U6.V+, U7.VDD, U8.VDD, U9.VDD; no longer JP1.1
- net V-: now also C14.1, JP4.2, U6.V-; no longer JP1.3
- net VAMP_PARA: now also JP2.1, U2.OUT_A; no longer JP2.2, U2.OUT_B
- net VBUFF: now also JP2.2, U2.+IN_A, U2.-IN_B, U2.OUT_B; no longer JP2.1, U2.+IN_B, U2.-IN_A, U2.OUT_A
- net VF_PARA: now also U2.-IN_A; no longer U2.-IN_B
- net VLOAD_PARA: now also JP5.1, U2.+IN_B; no longer U2.+IN_A
Other:
- note added: "DECIDE VALS"
- note added: "OUTPUT FOR TIA"
- note added: "SWITCHES FOR TIA"

Commit message: one mo' 'gin
Parts:
- added JP8: (no value), pinhead:PINHD-1X5/90
- added JP9: (no value), pinhead:PINHD-1X3/90
Connections:
- net AGND: now also JP8.5, JP9.3
- net SW1_TIA: now also JP8.1
- net SW2_TIA: now also JP8.2
- net SW3_TIA: now also JP8.3
- net SW4_TIA: now also JP8.4
- net VAMP_TIA: now also JP9.1
- net VOUT_TIA: now also JP9.2
Changed lines of the file:
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@@
 <setting verticaltext="up"/>
 </settings>
-<grid distance="0.1" unitdist="inch" unit="inch" style="lines" multiple="1" display="yes" altdistance="0.01" altunitdist="inch" altunit="inch"/>
+<grid distance="0.1" unitdist="inch" unit="inch" style="lines" multiple="1" display="no" altdistance="0.01" altunitdist="inch" altunit="inch"/>
 <layers>
 <layer number="1" name="Top" color="4" fill="1" visible="no" active="no"/>
@@
 <part name="C19" library="rcl" deviceset="C-EU" device="C0402" value="0.1uF"/>
 <part name="P+13" library="supply1" deviceset="V+" device=""/>
+<part name="JP8" library="pinhead" deviceset="PINHD-1X5" device="/90"/>
+<part name="AGND28" library="supply1" deviceset="AGND" device=""/>
+<part name="JP9" library="pinhead" deviceset="PINHD-1X3" device="/90"/>
+<part name="AGND29" library="supply1" deviceset="AGND" device=""/>
 </parts>
 <sheets>
@@
 <instance part="C19" gate="G$1" x="144.78" y="205.74" rot="R180"/>
 <instance part="P+13" gate="1" x="144.78" y="220.98"/>
+<instance part="JP8" gate="A" x="276.86" y="53.34"/>
+<instance part="AGND28" gate="VR1" x="264.16" y="43.18"/>
+<instance part="JP9" gate="A" x="210.82" y="50.8"/>
+<instance part="AGND29" gate="VR1" x="200.66" y="43.18"/>
 </instances>
 <busses>
@@
 <junction x="160.02" y="198.12"/>
 </segment>
+<segment>
+<pinref part="AGND28" gate="VR1" pin="AGND"/>
+<wire x1="264.16" y1="45.72" x2="264.16" y2="48.26" width="0.1524" layer="91"/>
+<pinref part="JP8" gate="A" pin="5"/>
+<wire x1="264.16" y1="48.26" x2="274.32" y2="48.26" width="0.1524" layer="91"/>
+</segment>
+<segment>
+<pinref part="JP9" gate="A" pin="3"/>
+<wire x1="208.28" y1="48.26" x2="200.66" y2="48.26" width="0.1524" layer="91"/>
+<wire x1="200.66" y1="48.26" x2="200.66" y2="45.72" width="0.1524" layer="91"/>
+<pinref part="AGND29" gate="VR1" pin="AGND"/>
+</segment>
 </net>
 <net name="V-" class="0">
@@
 <label x="144.78" y="76.2" size="1.778" layer="95"/>
 </segment>
+<segment>
+<pinref part="JP9" gate="A" pin="1"/>
+<wire x1="208.28" y1="53.34" x2="182.88" y2="53.34" width="0.1524" layer="91"/>
+<label x="175.26" y="53.34" size="1.778" layer="95"/>
+</segment>
 </net>
 <net name="VOUT_TIA" class="0">
@@
 <label x="45.72" y="78.74" size="1.778" layer="95"/>
 </segment>
+<segment>
+<pinref part="JP9" gate="A" pin="2"/>
+<wire x1="208.28" y1="50.8" x2="193.04" y2="50.8" width="0.1524" layer="91"/>
+<label x="190.5" y="50.8" size="1.778" layer="95"/>
+</segment>
 </net>
 <net name="VLOAD_TIA" class="0">
@@
 <label x="147.32" y="208.28" size="1.778" layer="95"/>
 </segment>
+<segment>
+<pinref part="JP8" gate="A" pin="1"/>
+<wire x1="274.32" y1="58.42" x2="254" y2="58.42" width="0.1524" layer="91"/>
+<label x="238.76" y="58.42" size="1.778" layer="95"/>
+</segment>
 </net>
 <net name="SOURCE_TIA" class="0">
@@
 <label x="147.32" y="127" size="1.778" layer="95"/>
 </segment>
+<segment>
+<pinref part="JP8" gate="A" pin="2"/>
+<wire x1="274.32" y1="55.88" x2="264.16" y2="55.88" width="0.1524" layer="91"/>
+<label x="248.92" y="55.88" size="1.778" layer="95"/>
+</segment>
 </net>
 <net name="SW3_TIA" class="0">
@@
 <label x="246.38" y="124.46" size="1.778" layer="95"/>
 </segment>
+<segment>
+<pinref part="JP8" gate="A" pin="3"/>
+<wire x1="274.32" y1="53.34" x2="254" y2="53.34" width="0.1524" layer="91"/>
+<label x="238.76" y="53.34" size="1.778" layer="95"/>
+</segment>
 </net>
 <net name="SW4_TIA" class="0">
@@
 <label x="337.82" y="124.46" size="1.778" layer="95"/>
 </segment>
-</net>
+<segment>
+<pinref part="JP8" gate="A" pin="4"/>
+<wire x1="274.32" y1="50.8" x2="264.16" y2="50.8" width="0.1524" layer="91"/>
+<label x="248.92" y="50.8" size="1.778" layer="95"/>
+</segment>
+</net>

Commit message: finished layout and board for z check
Parts:
- JP2: value (none) -> Droop_out
- JP3: value (none) -> Droop_sw
- JP7: value (none) -> Source_TIA
- JP8: value (none) -> TIA_sw
- JP9: value (none) -> TIA_out
- R1, R2, R3, R5, R6, R61, R62, R63, R64, R65: value (none) -> 2k
- R10, R11, R7, R8, R9: value (none) -> 20k
- R12, R13, R14, R15, R17, R4, R41, R42, R43, R44, R51, R52, R53, R54, R55: value (none) -> 200
- R16, R18, R20: value (none) -> 430
- R19: value (none) -> 510
- R21, R22, R23, R24: value (none) -> 750
- R25: value (none) -> 1000
- R26, R32, R33, R34, R35: value (none) -> 12k
- R27, R28, R29, R30, R31: value (none) -> 100
- R36, R37, R38, R39, R40: value (none) -> 300
- R46, R47, R48, R49, R50: value (none) -> 0
- R56, R57, R58, R59, R60: value (none) -> 1k
Connections:
- net SW1_TIA: now also U7.IN; no longer U10.IN
- net SW2_TIA: now also U8.IN; no longer U7.IN
- net SW3_TIA: now also U9.IN; no longer U8.IN
- net SW4_TIA: now also U10.IN; no longer U9.IN
Other:
- note added: "1k total"
- note added: "2k total"
- note added: "4k total"
- note added: "500 total"
- moved on the sheet: C11, C12, R10, R12, R13, R14, R15, R17, R18, R19, R2, R20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

Commit message: Finished layout and SS. Added gerbers
Parts:
- C1, C4: value 2.2uF -> 0.1uF
- C10, C7: value 0.1uF -> 2.2uF
- C12, C9: value 0.1uF -> 10nF
- C3, C6: value 10nF -> 0.1uF
- JP1: value PWR_IN -> Droop_out; device pinhead:PINHD-1X2/90 -> pinhead:PINHD-1X3/90
- JP2: value Droop_out -> Droop_sw; device pinhead:PINHD-1X3/90 -> pinhead:PINHD-1X5/90
- JP3: value Droop_sw -> Source; device pinhead:PINHD-1X5/90 -> pinhead:PINHD-1X1
- JP4: value PWR_IN -> Sink; device pinhead:PINHD-1X2/90 -> pinhead:PINHD-1X1
- JP5: value Source -> PWR_IN; device pinhead:PINHD-1X1 -> pinhead:PINHD-1X2/90
- JP6: value Sink -> PWR_IN; device pinhead:PINHD-1X1 -> pinhead:PINHD-1X2/90
- JP8: value TIA_sw -> TIA_out; device pinhead:PINHD-1X5/90 -> pinhead:PINHD-1X3/90
- JP9: value TIA_out -> TIA_sw; device pinhead:PINHD-1X3/90 -> pinhead:PINHD-1X5/90
- R1, R3, R5: value 2k -> 430
- R10, R7, R8, R9: value 20k -> 100
- R11: value 20k -> 200
- R16, R18: value 430 -> 750
- R17: value 200 -> 750
- R19: value 510 -> 750
- R2: value 2k -> 200
- R20: value 430 -> 1000
- R21, R22, R23, R24: value 750 -> 2k
- R25: value 1000 -> 2k
- R26: value 12k -> 20k
- R27, R28, R29, R30: value 100 -> 20k
- R31: value 100 -> 200
- R32, R33, R34, R35: value 12k -> 200
- R36, R37, R38, R39, R40: value 300 -> 12k
- R4: value 200 -> 510
- R41, R42, R43, R44: value 200 -> 300
- R45: value (none) -> 300
- R46, R47, R48, R49, R50: value 0 -> 2k
- R51, R52, R53, R54, R55: value 200 -> 0
- R56, R57, R58, R59, R60: value 1k -> 200
- R6: value 2k -> 100
- R61, R62, R63, R64, R65: value 2k -> 1k
- U2: value ADA4552-2ARM -> ADG801BRTZ-REEL7; device ScouseTomLib:ADA4552-2ARM -> Analog Devices_By_element14_Batch_1:ADG801BRTZ-REEL7
- U5: value ADG801BRTZ-REEL7 -> ADA4552-2ARM; device Analog Devices_By_element14_Batch_1:ADG801BRTZ-REEL7 -> ScouseTomLib:ADA4552-2ARM
Connections:
- removed net N$1 (its old number): R26.2, R32.2
- removed net N$24 (its old number): R25.2, U5.D
- removed net N$38 (its old number): R42.1, R43.1
- removed net N$39 (its old number): R43.2, R44.2
- removed net N$4 (its old number): R3.2, R5.2
- removed net N$40 (its old number): R44.1, R45.1
- removed net N$5 (its old number): R5.1, R6.1
- removed net N$7 (its old number): R7.2, R8.2
- removed net N$8 (its old number): R8.1, R9.1
- removed net N$9 (its old number): R10.2, R9.2
- new net N$17: R3.2, R4.2
- new net N$18: R4.1, R5.1
- new net N$19: R5.2, U1.D
- new net N$26: R6.2, R7.2
- new net N$27: R7.1, R8.1
- new net N$28: R8.2, R9.2
- new net N$33: R44.2, R45.2
- new net N$34: R43.1, R44.1
- new net N$35: R42.2, R43.2
- new net N$36: R41.1, R42.1
- net AGND: now also C1.1, C10.2, C11.2, C12.2, C2.1, C3.1, C4.1, C5.1, C7.2, C9.2, JP1.3, JP2.5, JP5.1, JP8.3, JP9.5, R30.1, R45.1, U2.GND, U2.NC, U2.S; no longer C1.2, C10.1, C11.1, C12.1, C2.2, C3.2, C4.2, C5.2, C7.1, C9.1, JP1.1, JP2.3, JP3.5, JP8.5, JP9.3, R36.1, R7.1, U5.GND, U5.NC, U5.S
- net N$10: now also R26.1, R27.1; no longer R10.1, R11.1
- net N$29: now also R10.1, R9.1; no longer R30.1, R31.1
- net N$31: now also R10.2, U2.D; no longer R31.2, U1.D
- net N$37: now also R31.2, R32.2; no longer R41.2, R42.2
- net N$6: now also R11.2; no longer R4.2
- net SW1_PARA: now also JP2.1, U2.IN; no longer JP3.1, U1.IN
- net SW1_TIA: now also JP9.1, U8.IN; no longer JP8.1, U7.IN
- net SW2_PARA: now also JP2.2; no longer JP3.2
- net SW2_TIA: now also JP9.2, U9.IN; no longer JP8.2, U8.IN
- net SW3_PARA: now also JP2.3, U1.IN; no longer JP3.3, U4.IN
- net SW3_TIA: now also JP9.3, U10.IN; no longer JP8.3, U9.IN
- net SW4_PARA: now also JP2.4, U4.IN; no longer JP3.4, U5.IN
- net SW4_TIA: now also JP9.4, U7.IN; no longer JP8.4, U10.IN
- net V+: now also C1.2, C2.2, C3.2, C4.2, C5.2, C7.1, C8.1, C9.1, JP5.2, U2.VDD, U5.V+; no longer C1.1, C10.2, C11.2, C12.2, C2.1, C3.1, C7.2, C9.2, JP1.2, U2.V+, U5.VDD
- net V-: now also C10.1, C11.1, C12.1, JP6.2, U5.V-; no longer C4.1, C5.1, C8.1, JP4.2, U2.V-
- net VAMP_PARA: now also JP1.1, R21.1, U5.OUT_A; no longer JP2.1, R1.1, U2.OUT_A
- net VAMP_TIA: now also JP8.1, R36.1; no longer JP9.1, R26.1
- net VBUFF: now also JP1.2, U5.+IN_A, U5.-IN_B, U5.OUT_B; no longer JP2.2, U2.+IN_A, U2.-IN_B, U2.OUT_B
- net VF_PARA: now also R25.2, R26.2, U5.-IN_A; no longer R11.2, R6.2, U2.-IN_A
- net VF_TIA: now also R41.2; no longer R35.2
- net VLOAD_PARA: now also JP3.1, R1.1, R11.1, R6.1, U5.+IN_B; no longer JP5.1, R21.1, R27.1, R4.1, U2.+IN_B
- net VLOAD_TIA: now also R31.1; no longer R41.1
- net VOUT_TIA: now also JP8.2, R35.2; no longer JP9.2, R45.2
Other:
- note added: "0 total"
- note added: "10k total"
- note added: "5k total"
- note removed: "DECIDE VALS"
- note removed: "OUTPUT FOR TIA"
- note removed: "SWITCHES FOR TIA"
