File: src/schematics/Output_Impedance_Tester/OutputZTester.brd (EAGLE design)
At the start: 160 x 100 mm, 0 parts

Commit message: Finished sim of TIA and Droop circuit. Started PCB
Parts:
- added C1, C4: 2.2uF, rcl:C0402
- added C10, C11, C12, C2, C5, C7, C8, C9: 0.1uF, rcl:C0402
- added C3, C6: 10nF, rcl:C0402
- added D1, D2: (no value), diode:DO-214AC
- added JP1: PWR_IN, pinhead:1X03/90
- added JP2: (no value), pinhead:1X03/90
- added R1, R10, R11, R12, R13, R14, R15, R16, R17, R18, R19, R2, R20, R21, R22, R23, R24, R25, R27, R28, R29, R3, R30, R31, R4, R5, R6, R7, R8, R9: (no value), rcl:R0402
- added TP1, TP2, TP3, TP4, TP5: TPSB1,27, testpad:B1,27
- added U1, U3, U4, U5: ADG801BRTZ-REEL7, Analog Devices_By_element14_Batch_1:SOT95P280X145-6N
- added U2: ADA4552-2ARM, ScouseTomLib:SOP65P490X110-8N
Connections:
- new net AGND: C1.2, C10.1, C11.1, C12.1, C2.2, C3.2, C4.2, C5.2, C6.2, C7.1, C8.2, C9.1, D1.A, D2.C, JP1.2, JP2.3, R7.1, U1.2, U1.3, U1.5, U3.2, U3.3, U3.5, U4.2, U4.3, U4.5, U5.2, U5.3, U5.5
- new net N$10: R10.1, R11.1
- new net N$11: R12.1, R13.1
- new net N$12: R13.2, R14.2
- new net N$13: R14.1, R15.1
- new net N$14: R15.2, U3.1
- new net N$15: R16.2, R17.2
- new net N$16: R17.1, R18.1
- new net N$17: R18.2, R19.2
- new net N$18: R19.1, R20.1
- new net N$19: R20.2, U4.1
- new net N$2: R1.2, R2.2
- new net N$20: R21.2, R22.2
- new net N$21: R22.1, R23.1
- new net N$22: R23.2, R24.2
- new net N$23: R24.1, R25.1
- new net N$24: R25.2, U5.1
- new net N$26: R27.2, R28.2
- new net N$27: R28.1, R29.1
- new net N$28: R29.2, R30.2
- new net N$29: R30.1, R31.1
- new net N$3: R2.1, R3.1
- new net N$31: R31.2, U1.1
- new net N$4: R3.2, R5.2
- new net N$5: R5.1, R6.1
- new net N$6: R12.2, R4.2
- new net N$7: R7.2, R8.2
- new net N$8: R8.1, R9.1
- new net N$9: R10.2, R9.2
- new net SW1_PARA: U1.4
- new net SW2_PARA: U3.4
- new net SW3_PARA: U4.4
- new net SW4_PARA: U5.4
- new net V+: C1.1, C10.2, C11.2, C12.2, C2.1, C3.1, C7.2, C9.2, D1.C, JP1.1, TP1.TP, U1.6, U2.8, U3.6, U4.6, U5.6
- new net V-: C4.1, C5.1, C6.1, C8.1, D2.A, JP1.3, TP2.TP, U2.4
- new net VAMP_PARA: JP2.2, R1.1, TP5.TP, U2.7
- new net VBUFF: JP2.1, TP4.TP, U2.1, U2.2, U2.5
- new net VF_PARA: R11.2, R6.2, U2.6
- new net VLOAD_PARA: R16.1, R21.1, R27.1, R4.1, TP3.TP, U2.3

Commit message: Basic layout for both circuits done
Parts:
- added C13, C14, C16, C17, C18, C19: 0.1uF, rcl:C0402
- added C15: 2.2nF, rcl:C0402
- added JP3: (no value), pinhead:1X05/90
- added JP4: PWR_IN, pinhead:1X02/90
- added JP5: Source, pinhead:1X01
- added JP6: Sink, pinhead:1X01
- added JP7: (no value), pinhead:1X01
- added R26, R32, R33, R34, R35, R36, R37, R38, R39, R40, R41, R42, R43, R44, R45, R46, R47, R48, R49, R50, R51, R52, R53, R54, R55, R56, R57, R58, R59, R60, R61, R62, R63, R64, R65: (no value), rcl:R0402
- added U10, U7, U8, U9: ADG801BRTZ-REEL7, Analog Devices_By_element14_Batch_1:SOT95P280X145-6N
- added U6: ADA4552-2ARM, ScouseTomLib:SOP65P490X110-8N
- D1, D2: value (none) -> 1N4148W-7-F; device diode:DO-214AC -> diode:SOD123
- JP1: device pinhead:1X03/90 -> pinhead:1X02/90
- moved TP5 255.7 mm to (44.5, 27.0), turned to 180 degrees
- moved TP2 251.7 mm to (44.5, 38.1)
- moved TP3 250.8 mm to (34.3, 34.3), turned to 270 degrees
- moved TP4 246.3 mm to (41.3, 23.2), turned to 180 degrees
- moved TP1 228.7 mm to (41.3, 20.3), turned to 180 degrees
- moved JP2 227.2 mm to (57.8, 24.1), turned to 270 degrees
- moved R24 225.5 mm to (24.1, 26.0)
- moved R21 224.9 mm to (24.8, 31.1), turned to 270 degrees
- moved R25 223.7 mm to (24.1, 24.8)
- moved R22 222.0 mm to (24.1, 28.6)
- moved R23 220.5 mm to (24.1, 27.3)
- moved C12 212.9 mm to (24.8, 18.4)
- moved U5 208.1 mm to (24.1, 21.6), turned to 270 degrees
- moved R19 207.0 mm to (27.9, 26.0)
- moved R16 206.3 mm to (28.6, 31.1), turned to 270 degrees
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Connections:
- new net N$1: R26.2, R32.2
- new net N$25: R32.1, R33.1
- new net N$30: R33.2, R34.2
- new net N$32: R34.1, R35.1
- new net N$33: R36.2, R37.2
- new net N$34: R37.1, R38.1
- new net N$35: R38.2, R39.2
- new net N$36: R39.1, R40.1
- new net N$37: R41.2, R42.2
- new net N$38: R42.1, R43.1
- new net N$39: R43.2, R44.2
- new net N$40: R44.1, R45.1
- new net N$41: R46.2, R47.2
- new net N$42: R47.1, R48.1
- new net N$43: R48.2, R49.2
- new net N$44: R49.1, R50.1
- new net N$46: R50.2, U7.2
- new net N$47: R51.2, R52.2
- new net N$48: R52.1, R53.1
- new net N$49: R53.2, R54.2
- new net N$50: R54.1, R55.1
- new net N$51: R55.2, U8.2
- new net N$52: R56.2, R57.2
- new net N$53: R57.1, R58.1
- new net N$54: R58.2, R59.2
- new net N$55: R59.1, R60.1
- new net N$56: R60.2, U9.2
- new net N$57: R61.2, R62.2
- new net N$58: R62.1, R63.1
- new net N$59: R63.2, R64.2
- new net N$60: R64.1, R65.1
- new net N$61: R65.2, U10.2
- new net SOURCE_TIA: JP7.1, U10.1, U7.1, U8.1, U9.1
- new net SW1_TIA: U10.4
- new net SW2_TIA: U7.4
- new net SW3_TIA: U8.4
- new net SW4_TIA: U9.4
- new net VAMP_TIA: R26.1, U6.1
- new net VF_TIA: R35.2, R40.2, U6.2
- new net VLOAD_TIA: C15.1, R41.1, R46.1, R51.1, R56.1, R61.1, U6.6
- new net VOUT_TIA: C15.2, R45.2, U6.3, U6.7
- net AGND: now also C13.1, C14.2, C16.1, C17.1, C18.1, C19.1, JP1.1, JP3.5, JP4.1, JP6.1, R36.1, U10.3, U10.5, U6.5, U7.3, U7.5, U8.3, U8.5, U9.3, U9.5; no longer JP1.2
- net SW1_PARA: now also JP3.1
- net SW2_PARA: now also JP3.2
- net SW3_PARA: now also JP3.3
- net SW4_PARA: now also JP3.4
- net V+: now also C13.2, C16.2, C17.2, C18.2, C19.2, JP1.2, U10.6, U6.8, U7.6, U8.6, U9.6; no longer JP1.1
- net V-: now also C14.1, JP4.2, U6.4; no longer JP1.3
- net VAMP_PARA: now also JP2.1, U2.1; no longer JP2.2, U2.7
- net VBUFF: now also JP2.2, U2.3, U2.6, U2.7; no longer JP2.1, U2.1, U2.2, U2.5
- net VF_PARA: now also U2.2; no longer U2.6
- net VLOAD_PARA: now also JP5.1, U2.5; no longer U2.3
Routing:
- net V+: track 0.00 -> 100.9 mm, vias 0 -> 4
- net AGND: track 0.00 -> 68.4 mm
- net VLOAD_TIA: track 0.00 -> 39.2 mm
- net V-: track 0.00 -> 27.6 mm
- net SOURCE_TIA: track 0.00 -> 26.8 mm
- net VLOAD_PARA: track 0.00 -> 25.8 mm
- net VBUFF: track 0.00 -> 23.4 mm
- net VAMP_PARA: track 0.00 -> 17.5 mm
- net VOUT_TIA: track 0.00 -> 11.3 mm
- net SW4_PARA: track 0.00 -> 8.15 mm, vias 0 -> 1
- net SW3_PARA: track 0.00 -> 7.62 mm, vias 0 -> 1
- net SW1_PARA: track 0.00 -> 7.62 mm, vias 0 -> 1
- net SW2_PARA: track 0.00 -> 7.10 mm, vias 0 -> 1
- net VF_PARA: track 0.00 -> 4.81 mm
- net VF_TIA: track 0.00 -> 3.64 mm
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
Commit message: one mo' 'gin
Parts:
- added JP8: (no value), pinhead:1X05/90
- added JP9: (no value), pinhead:1X03/90
- moved R36 1.63 mm to (37.5, 37.8), turned to 270 degrees
- moved C14 1.27 mm to (44.1, 31.7)
- moved R28 0.64 mm to (34.9, 28.6)
- moved R29 0.64 mm to (34.9, 27.3)
- moved R30 0.64 mm to (34.9, 26.0)
- moved R31 0.64 mm to (34.9, 24.8)
- moved R38 0.64 mm to (40.0, 36.8)
- moved U1 0.64 mm to (34.9, 21.6)
- moved R27 0.63 mm to (35.6, 31.1)
- moved R26 0.25 mm to (38.4, 30.5)
- moved R32 0.25 mm to (38.4, 31.8)
- moved R33 0.25 mm to (38.4, 33.0)
- moved R34 0.25 mm to (38.4, 34.3)
Connections:
- net AGND: now also JP8.5, JP9.3
- net SW1_TIA: now also JP8.1
- net SW2_TIA: now also JP8.2
- net SW3_TIA: now also JP8.3
- net SW4_TIA: now also JP8.4
- net VAMP_TIA: now also JP9.1
- net VOUT_TIA: now also JP9.2
Routing:
- net VOUT_TIA: track 11.3 -> 30.7 mm
- net VAMP_TIA: track 1.71 -> 16.7 mm
- net VLOAD_TIA: track 39.2 -> 34.7 mm
- net AGND: track 68.4 -> 63.9 mm
- net N$31: track 2.00 -> 0.00 mm
- net N$26: track 1.90 -> 0.00 mm
- net V+: track 100.9 -> 99.3 mm
- net V-: track 27.6 -> 26.9 mm

Commit message: finished layout and board for z check
Parts:
- JP2: value (none) -> Droop_out
- JP3: value (none) -> Droop_sw
- JP7: value (none) -> Source_TIA
- JP8: value (none) -> TIA_sw
- JP9: value (none) -> TIA_out
- R1, R2, R3, R5, R6, R61, R62, R63, R64, R65: value (none) -> 2k
- R10, R11, R7, R8, R9: value (none) -> 20k
- R12, R13, R14, R15, R17, R4, R41, R42, R43, R44, R51, R52, R53, R54, R55: value (none) -> 200
- R16, R18, R20: value (none) -> 430
- R19: value (none) -> 510
- R21, R22, R23, R24: value (none) -> 750
- R25: value (none) -> 1000
- R26, R32, R33, R34, R35: value (none) -> 12k
- R27, R28, R29, R30, R31: value (none) -> 100
- R36, R37, R38, R39, R40: value (none) -> 300
- R46, R47, R48, R49, R50: value (none) -> 0
- R56, R57, R58, R59, R60: value (none) -> 1k
- moved JP2 6.56 mm to (52.6, 20.1)
- moved C19 1.33 mm to (20.6, 24.1)
- moved C13 1.09 mm to (38.0, 26.9), turned to 180 degrees
- moved C18 0.40 mm to (20.6, 27.3)
Connections:
- net SW1_TIA: now also U7.4; no longer U10.4
- net SW2_TIA: now also U8.4; no longer U7.4
- net SW3_TIA: now also U9.4; no longer U8.4
- net SW4_TIA: now also U10.4; no longer U9.4
Routing:
- net AGND: track 63.9 -> 137.2 mm, vias 0 -> 12
- net SW4_TIA: track 0.00 -> 31.9 mm
- net SW3_TIA: track 0.00 -> 25.9 mm, vias 0 -> 1
- net SW2_TIA: track 0.00 -> 19.7 mm, vias 0 -> 1
- net V+: track 99.3 -> 113.1 mm, vias 4 -> 2
- net SW1_TIA: track 0.00 -> 11.4 mm, vias 0 -> 1
- net N$31: track 0.00 -> 2.17 mm
- net N$26: track 0.00 -> 1.91 mm
- net VAMP_TIA: track 16.7 -> 17.6 mm
- net VAMP_PARA: track 17.5 -> 16.9 mm
- added copper zone on layer 1, net AGND
- added copper zone on layer 16, net AGND
Other:
- board size 160 x 100 mm -> 38 x 34.6 mm

Commit message: Finished layout and SS. Added gerbers
Parts:
- C1, C4: value 2.2uF -> 0.1uF
- C10, C7: value 0.1uF -> 2.2uF
- C12, C9: value 0.1uF -> 10nF
- C3, C6: value 10nF -> 0.1uF
- JP1: value PWR_IN -> Droop_out; device pinhead:1X02/90 -> pinhead:1X03/90
- JP2: value Droop_out -> Droop_sw; device pinhead:1X03/90 -> pinhead:1X05/90
- JP3: value Droop_sw -> Source; device pinhead:1X05/90 -> pinhead:1X01
- JP4: value PWR_IN -> Sink; device pinhead:1X02/90 -> pinhead:1X01
- JP5: value Source -> PWR_IN; device pinhead:1X01 -> pinhead:1X02/90
- JP6: value Sink -> PWR_IN; device pinhead:1X01 -> pinhead:1X02/90
- JP8: value TIA_sw -> TIA_out; device pinhead:1X05/90 -> pinhead:1X03/90
- JP9: value TIA_out -> TIA_sw; device pinhead:1X03/90 -> pinhead:1X05/90
- R1, R3, R5: value 2k -> 430
- R10, R7, R8, R9: value 20k -> 100
- R11: value 20k -> 200
- R16, R18: value 430 -> 750
- R17: value 200 -> 750
- R19: value 510 -> 750
- R2: value 2k -> 200
- R20: value 430 -> 1000
- R21, R22, R23, R24: value 750 -> 2k
- R25: value 1000 -> 2k
- R26: value 12k -> 20k
- R27, R28, R29, R30: value 100 -> 20k
- R31: value 100 -> 200
- R32, R33, R34, R35: value 12k -> 200
- R36, R37, R38, R39, R40: value 300 -> 12k
- R4: value 200 -> 510
- R41, R42, R43, R44: value 200 -> 300
- R45: value (none) -> 300
- R46, R47, R48, R49, R50: value 0 -> 2k
- R51, R52, R53, R54, R55: value 200 -> 0
- R56, R57, R58, R59, R60: value 1k -> 200
- R6: value 2k -> 100
- R61, R62, R63, R64, R65: value 2k -> 1k
- U2: value ADA4552-2ARM -> ADG801BRTZ-REEL7; device ScouseTomLib:SOP65P490X110-8N -> Analog Devices_By_element14_Batch_1:SOT95P280X145-6N
- U5: value ADG801BRTZ-REEL7 -> ADA4552-2ARM; device Analog Devices_By_element14_Batch_1:SOT95P280X145-6N -> ScouseTomLib:SOP65P490X110-8N
- moved JP4 33.3 mm to (16.5, 22.9)
- moved JP5 33.3 mm to (41.3, 9.53), turned to 180 degrees
- moved JP6 33.3 mm to (41.3, 45.1)
- moved JP2 26.8 mm to (27.9, 9.53), turned to 180 degrees
- moved C12 26.2 mm to (41.3, 38.7), turned to 180 degrees
- moved R24 25.3 mm to (49.0, 30.8), turned to 270 degrees
- moved JP3 25.0 mm to (16.5, 31.8), turned to 0 degrees
- moved R23 24.8 mm to (49.0, 27.6), turned to 90 degrees
- moved R25 24.3 mm to (47.7, 30.8), turned to 270 degrees
- moved C4 24.3 mm to (24.8, 18.4), turned to 0 degrees
- moved R22 23.6 mm to (47.7, 27.6), turned to 90 degrees
- moved C11 22.9 mm to (41.3, 37.5), turned to 180 degrees
- moved R21 21.9 mm to (46.5, 28.4)
- moved R5 21.9 mm to (27.9, 24.8), turned to 0 degrees
- moved R3 21.0 mm to (27.9, 27.3), turned to 0 degrees
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Connections:
- removed net N$1 (its old number): R26.2, R32.2
- removed net N$24 (its old number): R25.2, U5.1
- removed net N$38 (its old number): R42.1, R43.1
- removed net N$39 (its old number): R43.2, R44.2
- removed net N$4 (its old number): R3.2, R5.2
- removed net N$40 (its old number): R44.1, R45.1
- removed net N$5 (its old number): R5.1, R6.1
- removed net N$7 (its old number): R7.2, R8.2
- removed net N$8 (its old number): R8.1, R9.1
- removed net N$9 (its old number): R10.2, R9.2
- new net N$17: R3.2, R4.2
- new net N$18: R4.1, R5.1
- new net N$19: R5.2, U1.1
- new net N$26: R6.2, R7.2
- new net N$27: R7.1, R8.1
- new net N$28: R8.2, R9.2
- new net N$33: R44.2, R45.2
- new net N$34: R43.1, R44.1
- new net N$35: R42.2, R43.2
- new net N$36: R41.1, R42.1
- net AGND: now also C1.1, C10.2, C11.2, C12.2, C2.1, C3.1, C4.1, C5.1, C7.2, C9.2, JP1.3, JP2.5, JP5.1, JP8.3, JP9.5, R30.1, R45.1, U2.2, U2.3, U2.5; no longer C1.2, C10.1, C11.1, C12.1, C2.2, C3.2, C4.2, C5.2, C7.1, C9.1, JP1.1, JP2.3, JP3.5, JP8.5, JP9.3, R36.1, R7.1, U5.2, U5.3, U5.5
- net N$10: now also R26.1, R27.1; no longer R10.1, R11.1
- net N$29: now also R10.1, R9.1; no longer R30.1, R31.1
- net N$31: now also R10.2, U2.1; no longer R31.2, U1.1
- net N$37: now also R31.2, R32.2; no longer R41.2, R42.2
- net N$6: now also R11.2; no longer R4.2
- net SW1_PARA: now also JP2.1, U2.4; no longer JP3.1, U1.4
- net SW1_TIA: now also JP9.1, U8.4; no longer JP8.1, U7.4
- net SW2_PARA: now also JP2.2; no longer JP3.2
- net SW2_TIA: now also JP9.2, U9.4; no longer JP8.2, U8.4
- net SW3_PARA: now also JP2.3, U1.4; no longer JP3.3, U4.4
- net SW3_TIA: now also JP9.3, U10.4; no longer JP8.3, U9.4
- net SW4_PARA: now also JP2.4, U4.4; no longer JP3.4, U5.4
- net SW4_TIA: now also JP9.4, U7.4; no longer JP8.4, U10.4
- net V+: now also C1.2, C2.2, C3.2, C4.2, C5.2, C7.1, C8.1, C9.1, JP5.2, U2.6, U5.8; no longer C1.1, C10.2, C11.2, C12.2, C2.1, C3.1, C7.2, C9.2, JP1.2, U2.8, U5.6
- net V-: now also C10.1, C11.1, C12.1, JP6.2, U5.4; no longer C4.1, C5.1, C8.1, JP4.2, U2.4
- net VAMP_PARA: now also JP1.1, R21.1, U5.1; no longer JP2.1, R1.1, U2.1
- net VAMP_TIA: now also JP8.1, R36.1; no longer JP9.1, R26.1
- net VBUFF: now also JP1.2, U5.3, U5.6, U5.7; no longer JP2.2, U2.3, U2.6, U2.7
- net VF_PARA: now also R25.2, R26.2, U5.2; no longer R11.2, R6.2, U2.2
- net VF_TIA: now also R41.2; no longer R35.2
- net VLOAD_PARA: now also JP3.1, R1.1, R11.1, R6.1, U5.5; no longer JP5.1, R21.1, R27.1, R4.1, U2.5
- net VLOAD_TIA: now also R31.1; no longer R41.1
- net VOUT_TIA: now also JP8.2, R35.2; no longer JP9.2, R45.2
Routing:
- net N$40 (its old number): track 2.16 -> 0.00 mm
- net N$24 (its old number): track 2.00 -> 0.00 mm
- net N$19: track 0.00 -> 2.00 mm
- net N$26: track 0.00 -> 1.91 mm
- net N$36: track 0.00 -> 1.90 mm
- net N$7 (its old number): track 1.88 -> 0.00 mm
- net N$4 (its old number): track 1.88 -> 0.00 mm
- net N$33: track 0.00 -> 1.64 mm
- net N$39 (its old number): track 1.53 -> 0.00 mm
- net N$38 (its old number): track 1.53 -> 0.00 mm
- net N$34: track 0.00 -> 1.52 mm
- net N$8 (its old number): track 1.28 -> 0.00 mm
- net N$35: track 0.00 -> 1.28 mm
- net N$9 (its old number): track 1.27 -> 0.00 mm
- net N$5 (its old number): track 1.27 -> 0.00 mm
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Other:
- board text added: "+5V"
- board text added: "-5V"
- board text added: "0"
- board text added: "10k"
- board text added: "1k"
- board text added: "2k"
- board text added: "4k"
- board text added: "500"
- board text added: "5k"
- board text added: "CS+"
- board text added: "CS-"
- board text added: "Droop Out"
- board text added: "Droop Switch"
- board text added: "G"
- board text added: "TIA Out"
- board text added: "TIA Switch"
- board text added: "Z CHK"
- board text added: "x1"
- board text added: "x10"
- board text added: "x40"
